Commit message: its working!

File: urdf/test_simple_arm.xacro.urdf (robot description, URDF)
Before this commit: robot arm, 3 links, 2 joints
Links:
- removed link lower_arm_link
- added link arm_base2_link, mass 0.01; visual cylinder length=0.01 radius=0.05
- added link arm_elbow_link, mass 0.01; visual cylinder length=${link_len} radius=0.01
- added link arm_shoulder_link, mass 0.01; visual cylinder length=${link_len} radius=0.01
- added link arm_wrist_link, mass 0.01; visual cylinder length=${wrist_len} radius=0.01
- link arm_base_link: mass 0.1 -> 0.01; geometry visual cylinder length=0.001 radius=0.05
Joints:
- removed joint joint_base
- added joint arm_base_joint: type continuous, parent arm_base_link, child arm_base2_link, origin xyz=0.0 0 0.002 rpy=0 0 0, axis 0 0 1, limit effort=1000.0 velocity=10
- added joint arm_elbow_joint: type continuous, parent arm_shoulder_link, child arm_elbow_link, origin xyz=0.0 0 ${link_len} rpy=0 0 0, axis 0 1 0, limit effort=1000.0 velocity=10
- added joint arm_shoulder_joint: type continuous, parent arm_base2_link, child arm_shoulder_link, origin xyz=0.0 0 0.01 rpy=0 0 0, axis 0 1 0, limit effort=1000.0 velocity=10
- added joint arm_wrist_joint: type continuous, parent arm_elbow_link, child arm_wrist_link, origin xyz=0.0 0 ${link_len} rpy=0 0 0, axis 0 1 0, limit effort=1000.0 velocity=10
